File: KicadJE_Counts3.sch (KiCad schematic (older format))
At the start: 57 parts, among them J301 ClockOut, J303 ClockIn, J304 Out0, J305 Out1, J306 Out2, J307 Out3, J308 Out4, J309 Out5, J310 Out6, J311 Out7, J312 Out8, J313 Out9, J314 Reset, P301 HEADER_2x5_Doepfer, SW301 Run

Commit message: counter fine
Parts:
- added C?: 47n, AJ:C_0805_AJ, symbol Device:C
- added D? (x2): 1N4007, Diode_SMD:D_MiniMELF, symbol Diode:LL4148
- added D?: 1N4148, Diode_SMD:D_MiniMELF, symbol Diode:LL4148
- added D?: LED_HLD, LED_THT:LED_D3.0mm, symbol Device:LED
- added J?: Hold, Connector_Audio:Jack_3.5mm_Ledino_KB3SPRS_Horizontal, symbol Connector:AudioJack2_SwitchT
- added R? (x10): 1k, Resistor_SMD:R_0805_2012Metric_Pad1.15x1.40mm_HandSolder, symbol Device:R
- added R? (x3): 10k, Resistor_SMD:R_0805_2012Metric_Pad1.15x1.40mm_HandSolder, symbol Device:R
- added R?: 100k, AJ:R_0805_AJ, symbol Device:R
- added R?: 10k, AJ:R_0805_AJ, symbol Device:R
- R301, R302, R303, R304, R306, R307, R310, R312, R313, R314, R315: value 4k7 -> 10k
Connections:
- net +12Vc: now also D?.1 (K), R?.1
- net ClockIn: now also R?.2; no longer U?.14 (CLK)
- net GNDS: now also C?.2, D?.1 (K), D?.2 (A), J?.S
- net Out0: now also R?.1; no longer U?.3 (Q0)
- net Out1: now also R?.1; no longer U?.2 (Q1)
- net Out2: now also R?.1; no longer U?.4 (Q2)
- net Out3: now also R?.1; no longer U?.7 (Q3)
- net Out4: now also R?.1; no longer U?.10 (Q4)
- net Out5: now also R?.1; no longer U?.1 (Q5)
- net Out6: now also R?.1; no longer U?.5 (Q6)
- net Out7: now also R?.1; no longer U?.6 (Q7)
- net Out8: now also R?.1; no longer U?.9 (Q8)
- net Out9: now also R?.1; no longer U?.11 (Q9)
- net OutCarry: now also R?.1; no longer SW301.3 (C)
- net Reset: now also R?.2; no longer U?.15 (Reset)
- new net: R?.2, U?.1 (Q5)
- new net: R?.2, U?.10 (Q4)
- new net: R?.2, U?.11 (Q9)
- new net: R?.1, U?.14 (CLK)
- new net: R?.1, U?.15 (Reset)
- new net: R?.2, U?.2 (Q1)
- new net: R?.2, U?.3 (Q0)
- new net: R?.2, U?.4 (Q2)
- new net: R?.2, U?.5 (Q6)
- new net: R?.2, U?.6 (Q7)
- new net: R?.2, U?.7 (Q3)
- new net: R?.2, U?.9 (Q8)
- new net: D?.2 (A), J?.T, R?.1
- new net: D?.2 (A), R?.2
- new net Hold: C?.1, D?.1 (K), D?.1 (K), D?.2 (A), R?.2, R?.2, SW301.3 (C)

Commit message: sch updates
Parts:
- removed D?: 1N4007, Diode_SMD:D_MiniMELF, symbol Diode:LL4148
- removed R?: 100k, AJ:R_0805_AJ, symbol Device:R
- added D?: LED_Clk_Out, LED_THT:LED_D3.0mm, symbol Device:LED
- added R?: 10k, Resistor_SMD:R_0805_2012Metric_Pad1.15x1.40mm_HandSolder, symbol Device:R
- D207: renamed from D302; value LED_Clk -> LED_Clk_In
- J214: renamed from J?; footprint Connector_Audio:Jack_3.5mm_Ledino_KB3SPRS_Horizontal -> AJ-Dropbox-Kicad:PJ301SM
- gave numbers to parts that had none: 26
- renumbered C309 to C201, C303 to C203, C304 to C204, C305 to C205, D301 to D201, D304 to D208, D305 to D209, D306 to D210, D307 to D211, D308 to D212, D309 to D213, D310 to D214, D311 to D215, D312 to D216, D313 to D217, D314 to D218, F301 to F201, J301 to J201, J303 to J202, J304 to J203, J305 to J204, J306 to J205, J307 to J206, J308 to J207, J309 to J208, J310 to J209, J311 to J210, J312 to J211, J313 to J212, J314 to J213, P301 to P201, R309 to R201, R308 to R202, R311 to R205, R301 to R219, R302 to R220, R303 to R221, R304 to R222, R305 to R223, R306 to R224, R307 to R225, R310 to R226, R312 to R227, R313 to R228, R314 to R229, R315 to R230, RV301 to RV201, SW301 to SW201
Connections:
- net ClockOut: now also R?.1
- net GNDS: now also D?.1 (K)
- net at R205.2, SW201.2 (B), U202.13 (CKEN): now also R231.1
- net at D221.2 (A), J214.T: no longer R231.1
- new net: D?.2 (A), R?.2
Other:
- moved on the sheet: D219, R231

Commit message: footprint updates
Parts:
- C201, C202, C204, C205: footprint Capacitor_SMD:C_0805_2012Metric_Pad1.15x1.40mm_HandSolder -> AJ:C_0805_AJ
- C203: footprint Capacitor_THT:CP_Radial_D5.0mm_P2.50mm -> Capacitor_SMD:C_1206_3216Metric
- D201: footprint Diode_SMD:D_SOD-123 -> AJ:D_SOD-123
- D202, D203, D204, D205: footprint Diode_THT:D_DO-41_SOD81_P10.16mm_Horizontal -> AJ:D_SOD-123
- D220, D221: footprint Diode_SMD:D_MiniMELF -> AJ:D_SOD-123
- R201, R202, R204, R205, R206, R207, R208, R209, R210, R211, R212, R213, R214, R215, R216, R217, R219, R220, R221, R222, R223, R224, R225, R226, R227, R228, R229, R230, R231: footprint Resistor_SMD:R_0805_2012Metric_Pad1.15x1.40mm_HandSolder -> AJ:R_0805_AJ
- R218: renamed from R?; footprint Resistor_SMD:R_0805_2012Metric_Pad1.15x1.40mm_HandSolder -> AJ:R_0805_AJ
- gave numbers to parts that had none: 1

Commit message: major components placed for counter
Parts:
- C203: value 100uF 16v -> 10uF 16v; symbol Device:CP -> Device:C
Changed lines of the file:
@@
 $EndComp
 $Comp
-L Device:CP C?
+L Device:C C?
 U 1 1 5C783FA4
 P 2150 1250
@@
 AR Path="/5C781441/5C783FA4" Ref="C203"  Part="1"
 F 0 "C203" H 2100 1450 50  0000 L CNN
-F 1 "100uF 16v" H 2000 1550 50  0000 L CNN
+F 1 "10uF 16v" H 2000 1550 50  0000 L CNN
 F 2 "Capacitor_SMD:C_1206_3216Metric" H 2188 1100 50  0001 C CNN
 F 3 "~" H 2150 1250 50  0001 C CNN

Commit message: Update KicadJE_Counts3.sch
Parts:
- R223: value 4k7 -> 10k
Changed lines of the file:
@@
 AR Path="/5C781441/5C83D871" Ref="R223"  Part="1"
 F 0 "R223" V 9668 2800 50  0000 C CNN
-F 1 "4k7" V 9759 2800 50  0000 C CNN
+F 1 "10k" V 9759 2800 50  0000 C CNN
 F 2 "AJ:R_0805_AJ" V 9805 2800 50  0001 C CNN
 F 3 "~" H 9875 2800 50  0001 C CNN
