File: KicadJE_Counts.kicad_pcb (KiCad board)
At the start: 2 copper layers, 242 x 128 mm, 218 parts, among them J101 Out1, J102 Out2, J103 In1.1, J104 In1.2, J105 In1.3, J106 In1.4, J201 Out2.1, J202 Out2.2, J203 In2.1, J204 CV2.1, J205 In2.2, J206 CV2.2, J301 In3.1, J302 Out3.1, J303 Out3.2, P101 HEADER_2x5_Doepfer, P201 HEADER_2x5_Doepfer, P301 HEADER_2x5_Doepfer, U101 TL072, U102 TL072, U201 TL072, U202 TL072, U301 TL072, U302 TL072

Commit message: Update KicadJE_Counts.kicad_pcb
Parts:
- removed C101, C102: 1u, Capacitor_SMD:C_1206_3216Metric_Pad1.42x1.75mm_HandSolder
- removed C103, C104, C105, C106: 100n, Capacitor_SMD:C_0805_2012Metric_Pad1.15x1.40mm_HandSolder
- removed C207, C212: OPEN, Capacitor_SMD:C_0805_2012Metric_Pad1.15x1.40mm_HandSolder
- removed C208, C209, C210: 1u, Capacitor_SMD:C_0805_2012Metric_Pad1.15x1.40mm_HandSolder
- removed C211: 4u7, Capacitor_SMD:C_0805_2012Metric_Pad1.15x1.40mm_HandSolder
- removed D101, D102, D104, D105, D106, D107, D108, D109, D110, D111: 1N1007, Diode_SMD:D_SOD-123
- removed D103: LED, LED_SMD:LED_0805_2012Metric_Pad1.15x1.40mm_HandSolder
- removed the D206 at (139.0, 118.5)
- removed the G*** at (132.0, 135.0)
- removed the G*** at (70.0, 135.0)
- removed the G*** at (102.0, 125.0)
- removed P101, P301: HEADER_2x5_Doepfer, Connector_IDC:IDC-Header_2x05_P2.54mm_Vertical
- removed R107, R108, R109, R110, R111, R112, R113, R114, R115, R116, R122, R123: 10k, Resistor_SMD:R_0805_2012Metric_Pad1.15x1.40mm_HandSolder
- removed R117: 100k, Resistor_SMD:R_0805_2012Metric_Pad1.15x1.40mm_HandSolder
- removed R118, R119, R120, R121, R128, R129: 20k, Resistor_SMD:R_0805_2012Metric_Pad1.15x1.40mm_HandSolder
- removed R124, R125, R130, R131: 1k, Resistor_SMD:R_0805_2012Metric_Pad1.15x1.40mm_HandSolder
- removed R126, R127: OPEN, Resistor_SMD:R_0805_2012Metric_Pad1.15x1.40mm_HandSolder
- removed the R218 at (134.5, 89.2)
- removed RV101: 100k Offset1, AJ-Dropbox-Kicad:Potentiometer_China_RK09_Single_Vertical_AJ
- removed RV102: 100k Gain1, AJ-Dropbox-Kicad:Potentiometer_China_RK09_Single_Vertical_AJ
- removed RV103: 100k Gain2, AJ-Dropbox-Kicad:Potentiometer_China_RK09_Single_Vertical_AJ
- removed RV104: 100k Offset2, AJ-Dropbox-Kicad:Potentiometer_China_RK09_Single_Vertical_AJ
- removed RV202: 100k Glide2, AJ-Dropbox-Kicad:Potentiometer_China_RK09_Single_Vertical_AJ
- removed TP111, TP209: Flow1, TestPoint:TestPoint_THTPad_2.0x2.0mm_Drill1.0mm
- removed the TP112 at (87.5, 104.0)
- removed TP210: Flow2, TestPoint:TestPoint_THTPad_2.0x2.0mm_Drill1.0mm
- removed U101, U102: TL072, AJ-Dropbox-Kicad:AJ_SO-8_5.3x6.2mm_P1.27mm
- added C311: 100n, AJ:C_0805_AJ, F.Cu at (89.8, 198.9)
- added C312: 100n, AJ:C_0805_AJ, F.Cu at (64.8, 222.3)
- added C313: 1u, AJ:C_0805_AJ, F.Cu at (98.4, 184.1)
- added C314: 1u, AJ:C_0805_AJ, F.Cu at (96.6, 187.1)
- added C315: 10n, AJ:C_0805_AJ, F.Cu at (91.8, 190.7)
- added C316: 1u, AJ:C_0805_AJ, F.Cu at (65.9, 219.3)
- added C317: 1u, AJ:C_0805_AJ, F.Cu at (80.7, 205.1)
- added C318: 1u, AJ:C_0805_AJ, F.Cu at (74.5, 209.6)
- added C319: 1u, AJ:C_0805_AJ, F.Cu at (85.0, 198.9)
- added C320: 10n, AJ:C_0805_AJ, F.Cu at (91.8, 187.7)
- added C321: 10n, AJ:C_0805_AJ, F.Cu at (80.7, 202.1)
- added C322: 10n, AJ:C_0805_AJ, F.Cu at (98.4, 181.2)
- added D206: 1N4007, Diode_SMD:D_MiniMELF, B.Cu at (135.1, 44.4)
- added D206: LED_Clk_Out, LED_THT:LED_D3.0mm, F.Cu at (116.2, 143.2)
- added D210: LED_2, LED_THT:LED_D3.0mm, F.Cu at (147.5, 125.0)
- added D211: LED_3, LED_THT:LED_D3.0mm, F.Cu at (147.5, 115.8)
- added D212: LED_4, LED_THT:LED_D3.0mm, F.Cu at (147.5, 106.5)
- added D213: LED_5, LED_THT:LED_D3.0mm, F.Cu at (147.5, 97.2)
- added D214: LED_6, LED_THT:LED_D3.0mm, F.Cu at (147.5, 88.2)
- added D215: LED_7, LED_THT:LED_D3.0mm, F.Cu at (147.5, 79.0)
- added D216: LED_8, LED_THT:LED_D3.0mm, F.Cu at (147.5, 69.8)
- added D217: LED_9, LED_THT:LED_D3.0mm, F.Cu at (147.8, 60.5)
- added D218: LED_RST, LED_THT:LED_D3.0mm, F.Cu at (116.5, 106.2)
- added D219: LED_HLD, LED_THT:LED_D3.0mm, F.Cu at (116.2, 115.2)
- added D220: 1N4007, AJ:D_SOD-123, B.Cu at (116.2, 18.2)
- added D221: 1N4148, AJ:D_SOD-123, B.Cu at (125.9, 30.0)
- added D309: LL4148, AJ:D_MiniMELF, F.Cu at (42.1, 225.5)
- added D310: LL4148, AJ:D_MiniMELF, F.Cu at (54.5, 219.8)
- added D311: LED, LED_THT:LED_D3.0mm, F.Cu at (67.9, 207.8)
- added D312: LED, LED_THT:LED_D3.0mm, F.Cu at (59.3, 217.7)
- added D313: LL4148, AJ:D_MiniMELF, F.Cu at (18.2, 225.8)
- added D314: LL4148, AJ:D_MiniMELF, F.Cu at (80.1, 195.7)
- added D315: LL4148, AJ:D_MiniMELF, F.Cu at (54.5, 216.6)
- added D316: LL4148, AJ:D_MiniMELF, F.Cu at (61.0, 213.3)
- added F201: Polyfuse, Fuse:Fuse_1206_3216Metric_Pad1.42x1.75mm_HandSolder, B.Cu at (141.2, 44.4)
- added F301: Polyfuse, Fuse:Fuse_1206_3216Metric_Pad1.42x1.75mm_HandSolder, F.Cu at (48.3, 225.5)
- added H301: 2,5mm, MountingHole:MountingHole_2.5mm_Pad_Via, F.Cu at (54.6, 211.7)
- added H302: 2,2mm, MountingHole:MountingHole_2.2mm_M2_Pad_Via, F.Cu at (86.5, 189.2)
- added H303: 2,5mm, MountingHole:MountingHole_2.5mm_Pad_Via, F.Cu at (86.8, 183.0)
- added H304: 2,2mm, MountingHole:MountingHole_2.2mm_M2_Pad_Via, F.Cu at (93.0, 182.7)
- added J107: Out6, AJ-Dropbox-Kicad:PJ301SM, F.Cu at (153.7, -70.4)
- added J207: Out4, AJ-Dropbox-Kicad:PJ301SM, F.Cu at (142.0, 108.2)
- added J208: Out5, AJ-Dropbox-Kicad:PJ301SM, F.Cu at (142.0, 99.0)
- added J209: Out6, AJ-Dropbox-Kicad:PJ301SM, F.Cu at (142.0, 89.8)
- added J210: Out7, AJ-Dropbox-Kicad:PJ301SM, F.Cu at (142.0, 80.6)
- added J211: Out8, AJ-Dropbox-Kicad:PJ301SM, F.Cu at (142.0, 71.4)
- added J212: Out9, AJ-Dropbox-Kicad:PJ301SM, F.Cu at (142.0, 62.2)
- added J213: Reset, AJ-Dropbox-Kicad:PJ301SM, F.Cu at (122.0, 108.0)
- added J214: Hold, AJ-Dropbox-Kicad:PJ301SM, F.Cu at (122.0, 117.0)
- added J304: Out 1, AJ-Dropbox-Kicad:PJ301SM, F.Cu at (78.4, 186.3)
- added J305: Out 2, AJ-Dropbox-Kicad:PJ301SM, F.Cu at (35.5, 215.0)
- added J306: Out 1 Final, AJ-Dropbox-Kicad:PJ301SM, F.Cu at (51.0, 200.6)
- added J307: Out 2 Final, AJ-Dropbox-Kicad:PJ301SM, F.Cu at (68.3, 186.3)
- added R218: 100k, AJ:R_0805_AJ, B.Cu at (131.4, 15.5)
- added R218: 10k, AJ:R_0805_AJ, F.Cu at (134.0, 155.0)
- added R230: 10k, AJ:R_0805_AJ, B.Cu at (112.5, 1.02)
- added R231: 10k, AJ:R_0805_AJ, B.Cu at (117.3, 4.27)
- added R325: 100k, AJ:R_0805_AJ, F.Cu at (74.3, 222.8)
- added R326: 10k, AJ:R_0805_AJ, F.Cu at (80.2, 216.9)
- added R327: 1k, AJ:R_0805_AJ, F.Cu at (88.7, 207.7)
- added R328: 1k, AJ:R_0805_AJ, F.Cu at (99.3, 196.6)
- added R329: 1k, AJ:R_0805_AJ, F.Cu at (75.4, 219.8)
- added R330: 1k, AJ:R_0805_AJ, F.Cu at (84.0, 208.0)
- added R331: 10R, AJ:R_0805_AJ, F.Cu at (79.2, 208.0)
- added R332: 1k, AJ:R_0805_AJ, F.Cu at (84.0, 211.0)
- added R333: 220R, AJ:R_0805_AJ, F.Cu at (68.9, 225.2)
- added RV303: 100k_A4, Potentiometer_THT:Potentiometer_China_RK09_Single_Vertical_AJ, F.Cu at (39.3, 189.4)
- added RV304: 100k_A4, Potentiometer_THT:Potentiometer_China_RK09_Single_Vertical_AJ, F.Cu at (32.1, 203.7)
- added SW201: Run, AJ-Dropbox-Kicad:SP1MS1, F.Cu at (122.0, 130.0)
- added U303: TL072, AJ-Dropbox-Kicad:AJ_SO-8_5.3x6.2mm_P1.27mm, F.Cu at (46.0, 220.0)
- added U304: TL072, AJ-Dropbox-Kicad:AJ_SO-8_5.3x6.2mm_P1.27mm, F.Cu at (71.6, 197.9)
- C201: value 1u -> 10n; footprint Capacitor_SMD:C_1206_3216Metric_Pad1.42x1.75mm_HandSolder -> AJ:C_0805_AJ; moved to B.Cu
- C202: value 1u -> 10u; footprint Capacitor_SMD:C_1206_3216Metric_Pad1.42x1.75mm_HandSolder -> AJ:C_0805_AJ; moved to B.Cu
- C203: value 100n -> 100uF 16v; footprint Capacitor_SMD:C_0805_2012Metric_Pad1.15x1.40mm_HandSolder -> Capacitor_SMD:C_1206_3216Metric
- C204, C205: footprint Capacitor_SMD:C_0805_2012Metric_Pad1.15x1.40mm_HandSolder -> AJ:C_0805_AJ
- C206: value 100n -> 47n; footprint Capacitor_SMD:C_0805_2012Metric_Pad1.15x1.40mm_HandSolder -> AJ:C_0805_AJ
- C301: value 1u -> 100n; footprint Capacitor_SMD:C_1206_3216Metric_Pad1.42x1.75mm_HandSolder -> AJ:C_0805_AJ
- C302: value 1u -> 100uF; footprint Capacitor_SMD:C_1206_3216Metric_Pad1.42x1.75mm_HandSolder -> Capacitor_SMD:C_1206_3216Metric
- C303, C304, C308: footprint Capacitor_SMD:C_0805_2012Metric_Pad1.15x1.40mm_HandSolder -> AJ:C_0805_AJ; moved to F.Cu
- C305, C306: value 100n -> 100uF 16v; footprint Capacitor_SMD:C_0805_2012Metric_Pad1.15x1.40mm_HandSolder -> Capacitor_SMD:C_1206_3216Metric; moved to F.Cu
- C307: value OPEN -> 100n; footprint Capacitor_SMD:C_0805_2012Metric_Pad1.15x1.40mm_HandSolder -> AJ:C_0805_AJ; moved to F.Cu
- C309, C310: value 1u -> 100n; footprint Capacitor_SMD:C_0805_2012Metric_Pad1.15x1.40mm_HandSolder -> AJ:C_0805_AJ; moved to F.Cu
- D201: footprint Diode_SMD:D_SOD-123 -> AJ:D_SOD-123; moved to B.Cu
- D202: value 1N1007 -> 1N5819; footprint Diode_SMD:D_SOD-123 -> AJ:D_SOD-123; moved to B.Cu
- D203: value LED -> 1N5819; footprint LED_SMD:LED_0805_2012Metric_Pad1.15x1.40mm_HandSolder -> AJ:D_SOD-123; moved to B.Cu
- D204: value 1N1007 -> 1N5819; footprint Diode_SMD:D_SOD-123 -> AJ:D_SOD-123
- D205: value LED -> 1N5819; footprint LED_THT:LED_D3.0mm -> AJ:D_SOD-123
- D207: value LED -> LED_Clk_In; moved to F.Cu
- D208: value 1N1007 -> LED_0; footprint Diode_SMD:D_SOD-123 -> LED_THT:LED_D3.0mm; moved to F.Cu
- D209: value 1N1007 -> LED_1; footprint Diode_SMD:D_SOD-123 -> LED_THT:LED_D3.0mm; moved to F.Cu
- D301, D302: footprint Diode_SMD:D_SOD-123 -> AJ:D_SOD-123
- D303: value LED -> 1N1007; footprint LED_SMD:LED_0805_2012Metric_Pad1.15x1.40mm_HandSolder -> AJ:D_SOD-123
- D304, D305: footprint Diode_SMD:D_SOD-123 -> AJ:D_SOD-123; moved to F.Cu
- D306: value 1N4148 -> 1N1007; footprint Diode_SMD:D_MiniMELF -> AJ:D_SOD-123; moved to F.Cu
- D307, D308: value 1N4148 -> LL4148; footprint Diode_SMD:D_MiniMELF -> AJ:D_MiniMELF; moved to F.Cu
- J101: value Out1 -> In7
- J102: value Out2 -> In6
- J103: value In1.1 -> In3
- J104: value In1.2 -> Out10
- J105: value In1.3 -> Out11
- J106: value In1.4 -> Out9
- J201: value Out2.1 -> ClockOut
- J202: value Out2.2 -> ClockIn
- J203: value In2.1 -> Out0
- J204: value CV2.1 -> Out1
- J205: value In2.2 -> Out2
- J206: value CV2.2 -> Out3
- J301: value In3.1 -> Doepfer connector; footprint AJ-Dropbox-Kicad:PJ301SM -> Connector_PinSocket_2.54mm:PinSocket_2x08_P2.54mm_Vertical
- J302: value Out3.1 -> In_1
- J303: value Out3.2 -> In 2
- P201: footprint Connector_IDC:IDC-Header_2x05_P2.54mm_Vertical -> Connector_PinHeader_2.54mm:PinHeader_2x05_P2.54mm_Vertical
- R101, R301: value 22k -> 10k; footprint Resistor_SMD:R_0805_2012Metric_Pad1.15x1.40mm_HandSolder -> AJ:R_0805_AJ
- R102, R103, R303, R323: value OPEN -> 10k; footprint Resistor_SMD:R_0805_2012Metric_Pad1.15x1.40mm_HandSolder -> AJ:R_0805_AJ; moved to F.Cu
- R104, R105: value 1k -> 10k; footprint Resistor_SMD:R_0805_2012Metric_Pad1.15x1.40mm_HandSolder -> AJ:R_0805_AJ; moved to F.Cu
- R106, R310: value 100k -> 10k; footprint Resistor_SMD:R_0805_2012Metric_Pad1.15x1.40mm_HandSolder -> AJ:R_0805_AJ; moved to F.Cu
- R201: value 22k -> 3k3; footprint Resistor_SMD:R_0805_2012Metric_Pad1.15x1.40mm_HandSolder -> AJ:R_0805_AJ; moved to B.Cu
- R202: value OPEN -> 220k; footprint Resistor_SMD:R_0805_2012Metric_Pad1.15x1.40mm_HandSolder -> AJ:R_0805_AJ
- R203, R224, R225: value OPEN -> 10k; footprint Resistor_SMD:R_0805_2012Metric_Pad1.15x1.40mm_HandSolder -> AJ:R_0805_AJ
- R204, R222: value 680R -> 10k; footprint Resistor_SMD:R_0805_2012Metric_Pad1.15x1.40mm_HandSolder -> AJ:R_0805_AJ
- R205: value 680R -> 47k; footprint Resistor_SMD:R_0805_2012Metric_Pad1.15x1.40mm_HandSolder -> AJ:R_0805_AJ
- R206, R207: footprint Resistor_SMD:R_0805_2012Metric_Pad1.15x1.40mm_HandSolder -> AJ:R_0805_AJ
- R208, R209, R210, R211: value 10k -> 1k; footprint Resistor_SMD:R_0805_2012Metric_Pad1.15x1.40mm_HandSolder -> AJ:R_0805_AJ
- R212, R213, R214, R215: value 20k -> 1k; footprint Resistor_SMD:R_0805_2012Metric_Pad1.15x1.40mm_HandSolder -> AJ:R_0805_AJ
- R216: value OPEN -> 1k; footprint OptoDevice:R_LDR_5.0x4.1mm_P3mm_Vertical -> AJ:R_0805_AJ
- R217: value LDR03_In2 -> 1k; footprint OptoDevice:R_LDR_5.0x4.1mm_P3mm_Vertical -> AJ:R_0805_AJ
- R219, R226, R227: value 20k -> 10k; footprint Resistor_SMD:R_0805_2012Metric_Pad1.15x1.40mm_HandSolder -> AJ:R_0805_AJ
- R220, R221: value 220R -> 10k; footprint Resistor_SMD:R_0805_2012Metric_Pad1.15x1.40mm_HandSolder -> AJ:R_0805_AJ
- R223: value 680R -> 4k7; footprint Resistor_SMD:R_0805_2012Metric_Pad1.15x1.40mm_HandSolder -> AJ:R_0805_AJ
- R228: value LDR03_In1 -> 10k; footprint OptoDevice:R_LDR_5.0x4.1mm_P3mm_Vertical -> AJ:R_0805_AJ
- R229: value OPEN -> 10k; footprint OptoDevice:R_LDR_5.0x4.1mm_P3mm_Vertical -> AJ:R_0805_AJ
- R302: value 10k -> OPEN; footprint Resistor_SMD:R_0805_2012Metric_Pad1.15x1.40mm_HandSolder -> AJ:R_0805_AJ; moved to F.Cu
- R304, R312, R315: footprint Resistor_SMD:R_0805_2012Metric_Pad1.15x1.40mm_HandSolder -> AJ:R_0805_AJ; moved to F.Cu
- R305: value 1k -> OPEN; footprint Resistor_SMD:R_0805_2012Metric_Pad1.15x1.40mm_HandSolder -> AJ:R_0805_AJ; moved to F.Cu
- R306: value 1k -> 100k; footprint Resistor_SMD:R_0805_2012Metric_Pad1.15x1.40mm_HandSolder -> AJ:R_0805_AJ; moved to F.Cu
- R307: value 47k -> 2k2; footprint Resistor_SMD:R_0805_2012Metric_Pad1.15x1.40mm_HandSolder -> AJ:R_0805_AJ; moved to F.Cu
- R308: value OPEN -> Open; footprint Resistor_SMD:R_0805_2012Metric_Pad1.15x1.40mm_HandSolder -> AJ:R_0805_AJ; moved to F.Cu
- R309, R314: value 220R -> 10k; footprint Resistor_SMD:R_0805_2012Metric_Pad1.15x1.40mm_HandSolder -> AJ:R_0805_AJ; moved to F.Cu
- R311: value 100k -> 0R; footprint Resistor_SMD:R_0805_2012Metric_Pad1.15x1.40mm_HandSolder -> AJ:R_0805_AJ; moved to F.Cu
- R313, R318: value OPEN -> 1k; footprint Resistor_SMD:R_0805_2012Metric_Pad1.15x1.40mm_HandSolder -> AJ:R_0805_AJ; moved to F.Cu
- R316: value 100k -> 1k; footprint Resistor_SMD:R_0805_2012Metric_Pad1.15x1.40mm_HandSolder -> AJ:R_0805_AJ; moved to F.Cu
- R317: value 220R -> 1k; footprint Resistor_SMD:R_0805_2012Metric_Pad1.15x1.40mm_HandSolder -> AJ:R_0805_AJ; moved to F.Cu
- R319: value OPEN -> 33k; footprint Resistor_SMD:R_0805_2012Metric_Pad1.15x1.40mm_HandSolder -> AJ:R_0805_AJ; moved to F.Cu
- R320: value 220R -> 100k; footprint Resistor_SMD:R_0805_2012Metric_Pad1.15x1.40mm_HandSolder -> AJ:R_0805_AJ; moved to F.Cu
- R321: value 20k -> Open; footprint Resistor_SMD:R_0805_2012Metric_Pad1.15x1.40mm_HandSolder -> AJ:R_0805_AJ; moved to F.Cu
- R322: value 20k -> 10k; footprint Resistor_SMD:R_0805_2012Metric_Pad1.15x1.40mm_HandSolder -> AJ:R_0805_AJ; moved to F.Cu
- R324: value OPEN -> 0R; footprint Resistor_SMD:R_0805_2012Metric_Pad1.15x1.40mm_HandSolder -> AJ:R_0805_AJ; moved to F.Cu
- RV201: value 100k Glide1 -> 50k_freq; footprint AJ-Dropbox-Kicad:Potentiometer_China_RK09_Single_Vertical_AJ -> Potentiometer_THT:Potentiometer_China_RK09_Single_Vertical_AJ
- RV301: value 100k PWM1 -> 100k_A4; footprint AJ-Dropbox-Kicad:Potentiometer_China_RK09_Single_Vertical_AJ -> Potentiometer_THT:Potentiometer_China_RK09_Single_Vertical_AJ
- RV302: value 100k PWM2 -> 100k_A4; footprint AJ-Dropbox-Kicad:Potentiometer_China_RK09_Single_Vertical_AJ -> Potentiometer_THT:Potentiometer_China_RK09_Single_Vertical_AJ
- U201: value TL072 -> LM555
- U202: value TL072 -> 4017; footprint AJ-Dropbox-Kicad:AJ_SO-8_5.3x6.2mm_P1.27mm -> Package_SO:SOIC-16_4.55x10.3mm_P1.27mm
- U301, U302: moved to F.Cu
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Connections:
- C201 pad 1: +12VA -> GNDS
- C201 pad 2: GND -> Net-(C201-Pad2)
- C202 pad 1: GND -> Net-(C202-Pad1)
- C202 pad 2: -12VA -> GNDS
- C203 pad 1: +12VA -> +12Vc
- C203 pad 2: GND -> GNDS
- C204 pad 1: GND -> GNDS
- C204 pad 2: -12VA -> +12Vc
- C205 pad 1: +12VA -> GNDS
- C205 pad 2: GND -> +12Vc
- C206 pad 1: GND -> Hold
- C206 pad 2: -12VA -> GNDS
- C301 pad 1: +12VA -> GND
- C301 pad 2: GND -> +5V
- C302 pad 1: GND -> +5V
- C302 pad 2: -12VA -> GND
- C303 pad 1: +12VA -> GND
- C303 pad 2: GND -> +12V
- C304 pad 1: GND -> -12V
- C304 pad 2: -12VA -> GND
- C305 pad 1: +12VA -> +12V
- C306 pad 2: -12VA -> -12V
- C307 pad 2: In3.1a -> +12V
- C308 pad 1: GND -> -12V
- C308 pad 2: Net-(C308-Pad2) -> GND
- C309 pad 2: Net-(C309-Pad2) -> +12V
- C310 pad 1: GND -> -12V
- C310 pad 2: Net-(C310-Pad2) -> GND
- D201 pad 1: +12VA -> +12Vc
- D201 pad 2: GND -> GNDS
- D202 pad 1: GND -> +12Vc
- D202 pad 2: -12VA -> ClockIn
- D203 pad 1: -12VA -> ClockIn
- D203 pad 2: Net-(D203-Pad2) -> GNDS
- D204 pad 1: +12VA -> +12Vc
- D204 pad 2: Net-(D204-Pad2) -> Reset
- D205 pad 1: GND -> Reset
- D205 pad 2: Net-(D205-Pad2) -> GNDS
- D207 pad 1: GND -> GNDS
- D208 pad 1: Net-(D204-Pad2) -> GNDS
- D208 pad 2: GND -> Net-(D208-Pad2)
- D209 pad 1: Net-(D206-Pad2) -> GNDS
- D209 pad 2: GND -> Net-(D209-Pad2)
- D301 pad 1: +12VA -> +12V
- D302 pad 2: -12VA -> -12V
- D303 pad 1: -12VA -> +12V
- D303 pad 2: Net-(D303-Pad2) -> Net-(C313-Pad1)
- D304 pad 1: +12VA -> Net-(C313-Pad1)
- D304 pad 2: Net-(D304-Pad2) -> -12V
- D305 pad 1: Net-(D304-Pad2) -> +12V
- D305 pad 2: GND -> Net-(C314-Pad1)
- D306 pad 1: In3.1a -> Net-(C314-Pad1)
- D306 pad 2: In3.1 -> -12V
- D307 pad 1: Net-(D307-Pad1) -> Net-(C315-Pad2)
- D307 pad 2: In3.1a -> Net-(C315-Pad1)
- D308 pad 1: In3.1a -> Net-(C315-Pad1)
- D308 pad 2: Net-(D308-Pad2) -> Net-(C315-Pad2)
- J103 pad TN: GND -> (no net)
- J104 pad T: Net-(J104-PadT) -> (no net)
- J104 pad TN: GND -> (no net)
- J105 pad T: Net-(J105-PadT) -> (no net)
- J105 pad TN: GND -> (no net)
- J106 pad T: Net-(J106-PadT) -> (no net)
- J106 pad TN: GND -> (no net)
- J201 pad S: GND -> GNDS
- J201 pad T: Net-(J201-PadT) -> ClockOut
- J202 pad S: GND -> GNDS
- J202 pad T: Net-(J202-PadT) -> ClockIn
- J202 pad TN: (no net) -> ClockOut
- J203 pad S: GND -> GNDS
- J203 pad T: Net-(J203-PadT) -> Out0
- J203 pad TN: GND -> (no net)
- J204 pad S: GND -> GNDS
- J204 pad T: Net-(J204-PadT) -> Out1
- J204 pad TN: GND -> (no net)
- J205 pad S: GND -> GNDS
- J205 pad T: Net-(J205-PadT) -> Out2
- J205 pad TN: GND -> (no net)
- J206 pad S: GND -> GNDS
- J206 pad T: Net-(J206-PadT) -> Out3
- J206 pad TN: GND -> (no net)
- J302 pad T: Net-(J302-PadT) -> Net-(C313-Pad1)
- J302 pad TN: (no net) -> Net-(C314-Pad1)
- J303 pad T: Net-(J303-PadT) -> Net-(C314-Pad1)
- J303 pad TN: (no net) -> Net-(J303-PadTN)
- P201 pad 1: -12VA -> /KicadJE_Counts3/-12
- P201 pad 10: +12VA -> /KicadJE_Counts3/+12
- P201 pad 2: -12VA -> /KicadJE_Counts3/-12
- P201 pad 3: GND -> GNDS
- P201 pad 4: GND -> GNDS
- P201 pad 5: GND -> GNDS
- P201 pad 6: GND -> GNDS
- P201 pad 7: GND -> GNDS
- P201 pad 8: GND -> GNDS
- P201 pad 9: +12VA -> /KicadJE_Counts3/+12
- R101 pad 1: Net-(D103-Pad2) -> Net-(J101-PadT)
- R101 pad 2: GND -> A7
- R102 pad 1: GND -> A7
- R102 pad 2: Net-(J101-PadT) -> GND
- R103 pad 1: GND -> Net-(J102-PadT)
- R103 pad 2: Net-(J102-PadT) -> A6
- R104 pad 1: Out1 -> A6
- R104 pad 2: Net-(J101-PadT) -> GND
- R105 pad 1: Out2 -> Net-(J103-PadT)
- R105 pad 2: Net-(J102-PadT) -> A3
- R106 pad 1: Net-(R106-Pad1) -> A3
- R106 pad 2: Out1 -> GND
- R201 pad 1: Net-(D203-Pad2) -> Net-(R201-Pad1)
- R201 pad 2: GND -> Net-(C202-Pad1)
- R202 pad 1: GND -> +12Vc
- R202 pad 2: Net-(J201-PadT) -> Net-(C202-Pad1)
- R203 pad 1: GND -> OutCarry
- R203 pad 2: Net-(J202-PadT) -> Hold
- R204 pad 2: Net-(J201-PadT) -> GNDS
- R205 pad 1: Net-(R205-Pad1) -> +12Vc
- R205 pad 2: Net-(J202-PadT) -> Net-(R205-Pad2)
- R206 pad 1: Net-(D204-Pad2) -> Net-(R206-Pad1)
- R206 pad 2: Net-(J203-PadT) -> ClockIn
- R207 pad 1: Net-(D205-Pad2) -> Net-(R207-Pad1)
- R207 pad 2: Net-(J204-PadT) -> Reset
- R208 pad 1: Net-(D206-Pad2) -> Out0
- R208 pad 2: Net-(J205-PadT) -> Net-(R208-Pad2)
- R209 pad 1: Net-(D207-Pad2) -> Out1
- R209 pad 2: Net-(J206-PadT) -> Net-(R209-Pad2)
- R210 pad 1: In2.1 -> Out2
- R210 pad 2: Net-(D204-Pad2) -> Net-(R210-Pad2)
- R211 pad 1: In2.2 -> Out3
- R211 pad 2: Net-(D206-Pad2) -> Net-(R211-Pad2)
- R212 pad 1: In2.1 -> Out4
- R212 pad 2: GND -> Net-(R212-Pad2)
- R213 pad 1: Net-(R213-Pad1) -> Out5
- R213 pad 2: GND -> Net-(R213-Pad2)
- R214 pad 1: In2.2 -> Out6
- R214 pad 2: GND -> Net-(R214-Pad2)
- R215 pad 1: Net-(R215-Pad1) -> Out7
- R215 pad 2: GND -> Net-(R215-Pad2)
- R216 pad 1: Net-(C207-Pad2) -> Out8
- R216 pad 2: Net-(R213-Pad1) -> Net-(R216-Pad2)
- R217 pad 1: Net-(C208-Pad2) -> Out9
- R217 pad 2: Net-(R215-Pad1) -> Net-(R217-Pad2)
- R219 pad 1: Net-(R213-Pad1) -> ClockIn
- R219 pad 2: Net-(C207-Pad1) -> Net-(D207-Pad2)
- R220 pad 1: Net-(R220-Pad1) -> Out0
- R220 pad 2: Net-(C207-Pad1) -> Net-(D208-Pad2)
- R221 pad 1: Net-(R221-Pad1) -> Out1
- R221 pad 2: Net-(C208-Pad1) -> Net-(D209-Pad2)
- R222 pad 1: Net-(R222-Pad1) -> Out2
- R222 pad 2: Net-(R220-Pad1) -> Net-(D210-Pad2)
- R223 pad 1: Net-(R223-Pad1) -> Out3
- R223 pad 2: Net-(R221-Pad1) -> Net-(D211-Pad2)
- R224 pad 1: Net-(C209-Pad1) -> Out4
- R224 pad 2: Net-(R222-Pad1) -> Net-(D212-Pad2)
- R225 pad 1: Net-(C210-Pad1) -> Out5
- R225 pad 2: Net-(R223-Pad1) -> Net-(D213-Pad2)
- R226 pad 1: Out2.1 -> Out6
- R226 pad 2: Net-(C209-Pad1) -> Net-(D214-Pad2)
- R227 pad 1: Net-(C210-Pad1) -> Out7
- R227 pad 2: Out2.2 -> Net-(D215-Pad2)
- R228 pad 1: Out2.1 -> Out8
- R229 pad 1: Net-(C212-Pad2) -> Out9
- R229 pad 2: Out2.2 -> Net-(D217-Pad2)
- R301 pad 1: Net-(D303-Pad2) -> Net-(C313-Pad2)
- R301 pad 2: GND -> In_1
- R302 pad 1: Net-(D304-Pad2) -> In_1
- R302 pad 2: Net-(J301-PadT) -> GND
- R303 pad 1: GND -> Net-(C314-Pad2)
- R303 pad 2: Net-(J302-PadT) -> In_2
- R304 pad 1: GND -> In_2
- R304 pad 2: Net-(J303-PadT) -> GND
- R305 pad 1: Out3.1 -> Net-(C313-Pad1)
- R305 pad 2: Net-(J302-PadT) -> Net-(J303-PadTN)
- R306 pad 1: Out3.2 -> Net-(C315-Pad1)
- R306 pad 2: Net-(J303-PadT) -> GND
- R307 pad 1: In3.1 -> /KicadJE_Counts2/POT1_L
- R307 pad 2: Net-(D304-Pad2) -> GND
- R308 pad 1: PosPk1 -> Net-(R308-Pad1)
- R308 pad 2: Net-(R308-Pad2) -> +12V
- R309 pad 1: NegPk1 -> Net-(C315-Pad1)
- R309 pad 2: Net-(R308-Pad2) -> In_2
- R310 pad 1: In3.1a -> Net-(R310-Pad1)
- R310 pad 2: GND -> In_1
- R311 pad 1: Out3.1 -> GND
- R311 pad 2: Net-(C308-Pad2) -> Net-(R308-Pad1)
- R312 pad 1: In3.1a -> GND
- R312 pad 2: Net-(R312-Pad2) -> Net-(R310-Pad1)
- R313 pad 1: +12VA -> (no net)
- R313 pad 2: Net-(R313-Pad2) -> Net-(C315-Pad1)
- R314 pad 1: GND -> /KicadJE_Counts2/POT3_C
- R314 pad 2: Net-(R313-Pad2) -> Net-(C315-Pad2)
- R315 pad 1: In3.1a -> Net-(C320-Pad2)
- R315 pad 2: Net-(R315-Pad2) -> /KicadJE_Counts2/POT1_C
- R316 pad 1: Net-(R312-Pad2) -> /KicadJE_Counts2/POT1_C
- R317 pad 1: Net-(R317-Pad1) -> /KicadJE_Counts2/POT3_C
- R317 pad 2: +12VA -> Out2_Dist
- R318 pad 1: Net-(R317-Pad1) -> Net-(R316-Pad2)
- R318 pad 2: GND -> Out1_Dist
- R319 pad 1: Net-(R319-Pad1) -> /KicadJE_Counts2/POT2_L
- R319 pad 2: NegPk1 -> GND
- R320 pad 1: Net-(R319-Pad1) -> Net-(R320-Pad1)
- R320 pad 2: PosPk1 -> GND
- R321 pad 1: Net-(D307-Pad1) -> Net-(R321-Pad1)
- R321 pad 2: Net-(C309-Pad2) -> +12V
- R322 pad 1: Net-(D308-Pad2) -> Net-(R320-Pad1)
- R322 pad 2: Net-(C310-Pad2) -> /KicadJE_Counts2/POT3_C
- R323 pad 1: PosPk1 -> Net-(R323-Pad1)
- R323 pad 2: Net-(C309-Pad2) -> Net-(R316-Pad2)
- R324 pad 1: NegPk1 -> GND
- R324 pad 2: Net-(C310-Pad2) -> Net-(R321-Pad1)
- RV201 pad 1: Net-(C209-Pad1) -> Net-(R201-Pad1)
- RV201 pad 2: Net-(R222-Pad1) -> ClockOut
- RV201 pad 3: Net-(R220-Pad1) -> ClockOut
- RV301 pad 1: Net-(R308-Pad2) -> (no net)
- RV301 pad 2: Net-(RV301-Pad2) -> /KicadJE_Counts2/POT3_C
- RV301 pad 3: Net-(R319-Pad1) -> /KicadJE_Counts2/POT3_H
- RV302 pad 1: Net-(R313-Pad2) -> /KicadJE_Counts2/POT4_L
- RV302 pad 2: Net-(R316-Pad2) -> /KicadJE_Counts2/POT4_C
- RV302 pad 3: Net-(R317-Pad1) -> /KicadJE_Counts2/POT4_H
- U201 pad 1: Net-(R204-Pad1) -> GNDS
- U201 pad 2: Net-(R204-Pad1) -> Net-(C202-Pad1)
- U201 pad 3: Out2.1 -> ClockOut
- U201 pad 4: -12VA -> +12Vc
- U201 pad 5: In2.1 -> Net-(C201-Pad2)
- U201 pad 6: Net-(R213-Pad1) -> Net-(C202-Pad1)
- U201 pad 7: Net-(C207-Pad1) -> (no net)
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Routing:
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Other:
- board text removed: "CV Util"
- board text removed: "TimeShift"

Commit message: major components placed for counter
Parts:
- removed the D206 at (135.1, 44.4)
- C203, D201, F201: moved to F.Cu
- R218: moved to B.Cu
- moved D220 95.4 mm to (120.5, 113.5), turned to 180 degrees
- moved J101 90.7 mm to (230.4, 7.58)
- moved J102 90.7 mm to (220.3, 21.9)
- moved J103 90.7 mm to (210.1, 21.9)
- moved J104 90.7 mm to (220.3, 7.58)
- moved J105 90.7 mm to (210.1, 7.58)
- moved J106 90.7 mm to (200.0, 21.9)
- moved J107 90.7 mm to (200.0, 7.58)
- moved R101 90.7 mm to (237.9, 2.48)
- moved R102 90.7 mm to (242.6, 2.48)
- moved R103 90.7 mm to (237.9, 5.43)
- moved R104 90.7 mm to (242.6, 5.43)
- moved R105 90.7 mm to (237.9, 8.38)
- moved R106 90.7 mm to (227.7, 16.8)
- moved U201 82.7 mm to (122.0, 75.0)
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
Commit message: Update KicadJE_Counts.kicad_pcb
Parts:
- moved R219 76.9 mm to (120.5, 102.0), turned to 180 degrees
- moved R206 61.5 mm to (124.7, 102.0), turned to 180 degrees
Changed lines of the file:
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@@
   )
   (module AJ:R_0805_AJ (layer B.Cu)
-    (at 146.575001 44.524999)
+    (at 124.674999 101.975001 180)
     (descr "Resistor SMD 0805 (2012 Metric), square (rectangular) end terminal, IPC_7351 nominal with elongated pad for handsoldering. (Body size source: https://docs.google.com/spreadsheets/d/1BsfQQcO9C6DZCsRaXUlFlo91Tg2WpOkGARC1WS5S8t0/edit?usp=sharing), generated with kicad-footprint-generator")
     (tags "resistor handsolder")
@@
     (fp_line (start -1 0.6) (end 1 0.6) (layer B.Fab) (width 0.1))
     (fp_line (start -1 -0.6) (end -1 0.6) (layer B.Fab) (width 0.1))
-    (pad 2 smd roundrect (at 1.025 0) (size 1.15 1.4) (layers B.Cu B.Paste B.Mask) (roundrect_rratio 0.217391)
+    (pad 2 smd roundrect (at 1.025 0 180) (size 1.15 1.4) (layers B.Cu B.Paste B.Mask) (roundrect_rratio 0.217391)
       (net 37 ClockIn))
-    (pad 1 smd roundrect (at -1.025 0) (size 1.15 1.4) (layers B.Cu B.Paste B.Mask) (roundrect_rratio 0.217391)
+    (pad 1 smd roundrect (at -1.025 0 180) (size 1.15 1.4) (layers B.Cu B.Paste B.Mask) (roundrect_rratio 0.217391)
       (net 75 "Net-(R206-Pad1)"))
     (model ${KISYS3DMOD}/Resistor_SMD.3dshapes/R_0805_2012Metric.wrl
@@
   )
   (module AJ:R_0805_AJ (layer B.Cu)
-    (at 154.005001 32.774999)
+    (at 120.5 102 180)
     (descr "Resistor SMD 0805 (2012 Metric), square (rectangular) end terminal, IPC_7351 nominal with elongated pad for handsoldering. (Body size source: https://docs.google.com/spreadsheets/d/1BsfQQcO9C6DZCsRaXUlFlo91Tg2WpOkGARC1WS5S8t0/edit?usp=sharing), generated with kicad-footprint-generator")
     (tags "resistor handsolder")
@@
       (effects (font (size 0.5 0.5) (thickness 0.08)) (justify mirror))
     )
-    (pad 1 smd roundrect (at -1.025 0) (size 1.15 1.4) (layers B.Cu B.Paste B.Mask) (roundrect_rratio 0.217391)
+    (pad 1 smd roundrect (at -1.025 0 180) (size 1.15 1.4) (layers B.Cu B.Paste B.Mask) (roundrect_rratio 0.217391)
       (net 37 ClockIn))
-    (pad 2 smd roundrect (at 1.025 0) (size 1.15 1.4) (layers B.Cu B.Paste B.Mask) (roundrect_rratio 0.217391)
+    (pad 2 smd roundrect (at 1.025 0 180) (size 1.15 1.4) (layers B.Cu B.Paste B.Mask) (roundrect_rratio 0.217391)
       (net 6 "Net-(D207-Pad2)"))
     (model ${KISYS3DMOD}/Resistor_SMD.3dshapes/R_0805_2012Metric.wrl

Commit message: Update KicadJE_Counts.kicad_pcb
Parts:
- moved R220 99.5 mm to (142.0, 141.0)
- moved C206 91.8 mm to (132.0, 120.5)
- moved R225 83.1 mm to (155.5, 95.0)
- moved R230 81.6 mm to (122.0, 108.0), turned to 180 degrees
- moved R207 80.1 mm to (132.0, 108.0), turned to 180 degrees
- moved R218 78.2 mm to (132.0, 104.5)
- moved R213 72.4 mm to (159.5, 95.0)
- moved R208 69.4 mm to (114.2, 86.8)
- moved R215 63.8 mm to (155.0, 74.8)
- moved R217 63.6 mm to (155.0, 66.2)
- moved R203 63.1 mm to (132.0, 102.0)
- moved R214 62.6 mm to (155.0, 89.2)
- moved R227 55.0 mm to (159.2, 74.5)
- moved R226 50.3 mm to (155.3, 86.0)
- moved R228 44.9 mm to (154.0, 70.5)
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
Commit message: Update KicadJE_Counts.kicad_pcb
Parts:
- moved C205 57.6 mm to (129.0, 89.5), turned to 180 degrees
- moved C204 48.9 mm to (129.0, 77.0), turned to 180 degrees
- moved R202 32.2 mm to (115.8, 74.8), turned to 270 degrees
- moved C202 27.3 mm to (115.8, 68.7), turned to 90 degrees
Changed lines of the file:
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@@
     (descr "LED, diameter 3.0mm, 2 pins")
     (tags "LED diameter 3.0mm 2 pins")
-    (fp_text reference D208 (at 1.27 -2.96 90) (layer F.SilkS)
+    (fp_text reference D208 (at 4.25 1.75 90) (layer F.SilkS)
       (effects (font (size 1 1) (thickness 0.15)))
     )
@@
     (descr "LED, diameter 3.0mm, 2 pins")
     (tags "LED diameter 3.0mm 2 pins")
-    (fp_text reference D209 (at 1.27 -2.96 90) (layer F.SilkS)
+    (fp_text reference D209 (at 4.5 1.5 90) (layer F.SilkS)
       (effects (font (size 1 1) (thickness 0.15)))
     )
@@
     (descr "LED, diameter 3.0mm, 2 pins")
     (tags "LED diameter 3.0mm 2 pins")
-    (fp_text reference D210 (at 1.27 -2.96 90) (layer F.SilkS)
+    (fp_text reference D210 (at 4.25 1.75 90) (layer F.SilkS)
       (effects (font (size 1 1) (thickness 0.15)))
     )
@@
     (descr "LED, diameter 3.0mm, 2 pins")
     (tags "LED diameter 3.0mm 2 pins")
-    (fp_text reference D211 (at 1.27 -2.96 90) (layer F.SilkS)
+    (fp_text reference D211 (at 4.25 1.75 90) (layer F.SilkS)
       (effects (font (size 1 1) (thickness 0.15)))
     )
@@
     (descr "LED, diameter 3.0mm, 2 pins")
     (tags "LED diameter 3.0mm 2 pins")
-    (fp_text reference D212 (at 1.27 -2.96 90) (layer F.SilkS)
+    (fp_text reference D212 (at 4.25 1.75 90) (layer F.SilkS)
       (effects (font (size 1 1) (thickness 0.15)))
     )
@@
     (descr "LED, diameter 3.0mm, 2 pins")
     (tags "LED diameter 3.0mm 2 pins")
-    (fp_text reference D213 (at 2 -4.75 90) (layer F.SilkS)
+    (fp_text reference D213 (at 4.25 1.75 90) (layer F.SilkS)
       (effects (font (size 1 1) (thickness 0.15)))
     )
@@
     (descr "LED, diameter 3.0mm, 2 pins")
     (tags "LED diameter 3.0mm 2 pins")
-    (fp_text reference D214 (at 1.27 -2.96 90) (layer F.SilkS)
+    (fp_text reference D214 (at 4.5 1.75 90) (layer F.SilkS)
       (effects (font (size 1 1) (thickness 0.15)))
     )
@@
     (descr "LED, diameter 3.0mm, 2 pins")
     (tags "LED diameter 3.0mm 2 pins")
-    (fp_text reference D215 (at 1.27 -2.96 90) (layer F.SilkS)
+    (fp_text reference D215 (at 4.5 1.75 90) (layer F.SilkS)
       (effects (font (size 1 1) (thickness 0.15)))
     )
@@
     (descr "LED, diameter 3.0mm, 2 pins")
     (tags "LED diameter 3.0mm 2 pins")
-    (fp_text reference D216 (at 1.27 -2.96 90) (layer F.SilkS)
+    (fp_text reference D216 (at 4.25 1.75 90) (layer F.SilkS)
       (effects (font (size 1 1) (thickness 0.15)))
     )
@@
     (descr "LED, diameter 3.0mm, 2 pins")
     (tags "LED diameter 3.0mm 2 pins")
-    (fp_text reference D217 (at 1.27 -2.96 90) (layer F.SilkS)
+    (fp_text reference D217 (at 4.75 1.75 90) (layer F.SilkS)
       (effects (font (size 1 1) (thickness 0.15)))
     )
@@
       (effects (font (size 0.75 1) (thickness 0.125)))
     )
-    (fp_text value ClockOut (at 3 5.5 90) (layer F.SilkS)
+    (fp_text value ClockOut (at 0 -7.5 90) (layer F.SilkS)
       (effects (font (size 1 1) (thickness 0.15)))
     )
@@
       (effects (font (size 0.75 1) (thickness 0.125)))
     )
-    (fp_text value ClockIn (at 3 5.5 90) (layer F.SilkS)
+    (fp_text value ClockIn (at 0 -6.75 90) (layer F.SilkS)
       (effects (font (size 1 1) (thickness 0.15)))
     )
@@
       (effects (font (size 0.75 1) (thickness 0.125)))
     )
-    (fp_text value Reset (at 3 5.5 90) (layer F.SilkS)
+    (fp_text value Reset (at 0 -6.75 90) (layer F.SilkS)
       (effects (font (size 1 1) (thickness 0.15)))
     )
@@
       (effects (font (size 0.75 1) (thickness 0.125)))
     )
-    (fp_text value Hold (at 3 5.5 90) (layer F.SilkS)
+    (fp_text value Hold (at 0 -7 90) (layer F.SilkS)
       (effects (font (size 1 1) (thickness 0.15)))
     )
@@
   )
   (module AJ:C_0805_AJ (layer B.Cu)
-    (at 124.75 43)
+    (at 115.75 68.725 90)
     (descr "Capacitor SMD 0805 (2012 Metric), square (rectangular) end terminal, IPC_7351 nominal with elongated pad for handsoldering. (Body size source: https://docs.google.com/spreadsheets/d/1BsfQQcO9C6DZCsRaXUlFlo91Tg2WpOkGARC1WS5S8t0/edit?usp=sharing), generated with kicad-footprint-generator")
     (tags "capacitor handsolder")
     (attr smd)
-    (fp_text reference C202 (at -3.975 0) (layer B.SilkS)
+    (fp_text reference C202 (at 3.975 -1 90) (layer B.SilkS)
       (effects (font (size 1 1) (thickness 0.15)) (justify mirror))
     )
-    (fp_text value 10u (at 0 -1.65) (layer B.SilkS)
+    (fp_text value 10u (at -3.025 -1 90) (layer B.SilkS)
       (effects (font (size 0.8 0.8) (thickness 0.1)) (justify mirror))
     )
-    (fp_text user %R (at 0 0) (layer B.Fab)
+    (fp_text user %R (at 0 0 90) (layer B.Fab)
       (effects (font (size 0.5 0.5) (thickness 0.08)) (justify mirror))
     )
@@
     (fp_line (start -1 0.6) (end 1 0.6) (layer B.Fab) (width 0.1))
     (fp_line (start -1 -0.6) (end -1 0.6) (layer B.Fab) (width 0.1))
-    (pad 2 smd roundrect (at 1.025 0) (size 1.15 1.4) (layers B.Cu B.Paste B.Mask) (roundrect_rratio 0.217391)
+    (pad 2 smd roundrect (at 1.025 0 90) (size 1.15 1.4) (layers B.Cu B.Paste B.Mask) (roundrect_rratio 0.217391)
       (net 12 GNDS))
-    (pad 1 smd roundrect (at -1.025 0) (size 1.15 1.4) (layers B.Cu B.Paste B.Mask) (roundrect_rratio 0.217391)
+    (pad 1 smd roundrect (at -1.025 0 90) (size 1.15 1.4) (layers B.Cu B.Paste B.Mask) (roundrect_rratio 0.217391)
       (net 13 "Net-(C202-Pad1)"))
     (model ${KISYS3DMOD}/Capacitor_SMD.3dshapes/C_0805_2012Metric.wrl
@@
   )
   (module AJ:C_0805_AJ (layer B.Cu)
-    (at 113 30.75)
+    (at 129 77 180)
     (descr "Capacitor SMD 0805 (2012 Metric), square (rectangular) end terminal, IPC_7351 nominal with elongated pad for handsoldering. (Body size source: https://docs.google.com/spreadsheets/d/1BsfQQcO9C6DZCsRaXUlFlo91Tg2WpOkGARC1WS5S8t0/edit?usp=sharing), generated with kicad-footprint-generator")
     (tags "capacitor handsolder")
@@
       (effects (font (size 0.5 0.5) (thickness 0.08)) (justify mirror))
     )
-    (pad 1 smd roundrect (at -1.025 0) (size 1.15 1.4) (layers B.Cu B.Paste B.Mask) (roundrect_rratio 0.217391)
+    (pad 1 smd roundrect (at -1.025 0 180) (size 1.15 1.4) (layers B.Cu B.Paste B.Mask) (roundrect_rratio 0.217391)
       (net 12 GNDS))
-    (pad 2 smd roundrect (at 1.025 0) (size 1.15 1.4) (layers B.Cu B.Paste B.Mask) (roundrect_rratio 0.217391)
+    (pad 2 smd roundrect (at 1.025 0 180) (size 1.15 1.4) (layers B.Cu B.Paste B.Mask) (roundrect_rratio 0.217391)
       (net 14 +12Vc))
     (model ${KISYS3DMOD}/Capacitor_SMD.3dshapes/C_0805_2012Metric.wrl
@@
   )
   (module AJ:C_0805_AJ (layer B.Cu)
-    (at 113.075001 34.124999)
+    (at 129 89.5 180)
     (descr "Capacitor SMD 0805 (2012 Metric), square (rectangular) end terminal, IPC_7351 nominal with elongated pad for handsoldering. (Body size source: https://docs.google.com/spreadsheets/d/1BsfQQcO9C6DZCsRaXUlFlo91Tg2WpOkGARC1WS5S8t0/edit?usp=sharing), generated with kicad-footprint-generator")
     (tags "capacitor handsolder")
@@
     (fp_line (start -1 0.6) (end 1 0.6) (layer B.Fab) (width 0.1))
     (fp_line (start -1 -0.6) (end -1 0.6) (layer B.Fab) (width 0.1))
-    (pad 2 smd roundrect (at 1.025 0) (size 1.15 1.4) (layers B.Cu B.Paste B.Mask) (roundrect_rratio 0.217391)
+    (pad 2 smd roundrect (at 1.025 0 180) (size 1.15 1.4) (layers B.Cu B.Paste B.Mask) (roundrect_rratio 0.217391)
       (net 14 +12Vc))
-    (pad 1 smd roundrect (at -1.025 0) (size 1.15 1.4) (layers B.Cu B.Paste B.Mask) (roundrect_rratio 0.217391)
+    (pad 1 smd roundrect (at -1.025 0 180) (size 1.15 1.4) (layers B.Cu B.Paste B.Mask) (roundrect_rratio 0.217391)
       (net 12 GNDS))
     (model ${KISYS3DMOD}/Capacitor_SMD.3dshapes/C_0805_2012Metric.wrl
@@
   )
   (module AJ:R_0805_AJ (layer B.Cu)
-    (at 120.575001 42.884999)
+    (at 115.75 74.75 270)
     (descr "Resistor SMD 0805 (2012 Metric), square (rectangular) end terminal, IPC_7351 nominal with elongated pad for handsoldering. (Body size source: https://docs.google.com/spreadsheets/d/1BsfQQcO9C6DZCsRaXUlFlo91Tg2WpOkGARC1WS5S8t0/edit?usp=sharing), generated with kicad-footprint-generator")
     (tags "resistor handsolder")
     (attr smd)
-    (fp_text reference R202 (at 0 1.65) (layer B.SilkS)
+    (fp_text reference R202 (at 3.75 -0.5 90) (layer B.SilkS)
       (effects (font (size 1 1) (thickness 0.15)) (justify mirror))
     )
-    (fp_text value 220k (at 0 -1.65) (layer B.SilkS)
+    (fp_text value 220k (at 3.5 1 90) (layer B.SilkS)
       (effects (font (size 0.8 0.8) (thickness 0.1)) (justify mirror))
     )
@@
     (fp_line (start 1.85 0.95) (end 1.85 -0.95) (layer B.CrtYd) (width 0.05))
     (fp_line (start 1.85 -0.95) (end -1.85 -0.95) (layer B.CrtYd) (width 0.05))
-    (fp_text user %R (at 0 0) (layer B.Fab)
+    (fp_text user %R (at 0 0 90) (layer B.Fab)
       (effects (font (size 0.5 0.5) (thickness 0.08)) (justify mirror))
     )
-    (pad 1 smd roundrect (at -1.025 0) (size 1.15 1.4) (layers B.Cu B.Paste B.Mask) (roundrect_rratio 0.217391)
+    (pad 1 smd roundrect (at -1.025 0 270) (size 1.15 1.4) (layers B.Cu B.Paste B.Mask) (roundrect_rratio 0.217391)
       (net 14 +12Vc))
-    (pad 2 smd roundrect (at 1.025 0) (size 1.15 1.4) (layers B.Cu B.Paste B.Mask) (roundrect_rratio 0.217391)
+    (pad 2 smd roundrect (at 1.025 0 270) (size 1.15 1.4) (layers B.Cu B.Paste B.Mask) (roundrect_rratio 0.217391)
       (net 13 "Net-(C202-Pad1)"))
     (model ${KISYS3DMOD}/Resistor_SMD.3dshapes/R_0805_2012Metric.wrl

Commit message: Count routed w component labels
Parts:
- C203, D201, F201: moved to B.Cu
- moved R221 101.1 mm to (142.0, 131.5)
- moved R209 100.1 mm to (137.8, 131.5), turned to 180 degrees
- moved R204 98.3 mm to (132.0, 130.0)
- moved R222 96.6 mm to (142.0, 122.5)
- moved R210 95.6 mm to (137.8, 122.5), turned to 180 degrees
- moved R223 91.7 mm to (142.0, 113.2)
- moved R211 90.6 mm to (137.8, 113.2), turned to 180 degrees
- moved R205 87.9 mm to (125.8, 112.8), turned to 180 degrees
- moved R231 84.5 mm to (122.0, 112.8), turned to 180 degrees
- moved R212 60.8 mm to (137.8, 103.9), turned to 180 degrees
- moved R208 58.9 mm to (137.7, 140.8), turned to 180 degrees
- moved R224 58.2 mm to (142.2, 103.9)
- moved C201 33.6 mm to (129.0, 73.0), turned to 180 degrees
- moved R216 22.1 mm to (137.8, 67.2), turned to 180 degrees
- moved R213 21.8 mm to (137.8, 94.8), turned to 180 degrees
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Routing:
- net ClockOut: track 0.00 -> 117.5 mm
- net +12Vc: track 0.00 -> 94.1 mm, vias 0 -> 6
- net Net-(R205-Pad2): track 0.00 -> 71.5 mm, vias 0 -> 2
- net Net-(R208-Pad2): track 0.00 -> 62.9 mm
- net GNDS: track 0.00 -> 59.6 mm, vias 0 -> 37
- net Net-(R209-Pad2): track 0.00 -> 57.9 mm
- net Net-(R210-Pad2): track 0.00 -> 45.9 mm
- net Hold: track 0.00 -> 42.9 mm
- net Net-(R211-Pad2): track 0.00 -> 40.7 mm
- net Net-(R217-Pad2): track 0.00 -> 37.3 mm
- net Net-(R212-Pad2): track 0.00 -> 29.7 mm
- net Net-(R207-Pad1): track 0.00 -> 29.0 mm, vias 0 -> 2
- net Net-(R215-Pad2): track 0.00 -> 25.1 mm
- net OutCarry: track 0.00 -> 24.8 mm, vias 0 -> 2
- net Net-(C202-Pad1): track 0.00 -> 24.8 mm
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- added copper zone on B.Cu, net GNDS
- added copper zone on F.Cu, net GNDS

Commit message: Update KicadJE_Counts.kicad_pcb
Count labels
Parts:
- added G***: LOGO, AJ:Johansen_engineering_logo_20mm, F.Cu at (122.0, 136.0)
Other:
- board text added: "COUNT RevB"
- board text added: "Johansen Engineering Count Rev B 05/05-2020"

Commit message: Update KicadJE_Counts.kicad_pcb
Parts:
- removed C301, C303, C304, C307, C308: 100n, AJ:C_0805_AJ
- removed C302: 100uF, Capacitor_SMD:C_1206_3216Metric
- removed F301: Polyfuse, Fuse:Fuse_1206_3216Metric_Pad1.42x1.75mm_HandSolder
- removed U303, U304: TL072, AJ-Dropbox-Kicad:AJ_SO-8_5.3x6.2mm_P1.27mm
- C203: value 100uF 16v -> 10uF 16v
- C305, C306, C309, C310, C311, C312, C313, C314, C315, C316, C317, C318, C319, C320, C321, C322, D301, D302, D303, D304, D305, D306, D307, D308, D309, D310, D313, D314, D315, D316, H301, H302, H303, H304, J301, R301, R302, R303, R304, R305, R306, R307, R308, R309, R310, R311, R312, R313, R314, R315, R316, R317, R318, R319, R320, R321, R322, R323, R324, R325, R326, R327, R328, R329, R330, R331, R332, R333, U301, U302: moved to B.Cu
- R223: value 4k7 -> 10k
- moved J301 138.2 mm to (68.7, 52.8), turned to 180 degrees
- moved J305 59.9 mm to (85.0, 181.2)
- moved RV301 59.9 mm to (66.2, 178.0)
- moved C306 56.2 mm to (83.8, 231.9)
- moved H303 54.7 mm to (59.2, 230.2)
- moved D311 50.6 mm to (37.2, 167.5)
- moved C322 49.9 mm to (82.9, 228.7)
- moved J303 46.4 mm to (103.4, 181.4)
- moved J306 46.4 mm to (93.2, 181.4)
- moved H304 46.3 mm to (54.6, 208.5)
- moved D312 44.0 mm to (44.0, 176.5)
- moved C313 41.9 mm to (65.7, 210.4)
- moved C315 41.5 mm to (88.9, 232.0)
- moved D313 41.1 mm to (59.1, 222.1)
- moved H302 40.8 mm to (71.8, 227.3)
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Connections:
- J301 pad 5: /KicadJE_Counts2/+5Vin -> +5V
- J301 pad 6: /KicadJE_Counts2/+5Vin -> +5V
