File: KicadJE_Counts2.sch (KiCad schematic (older format))
At the start: 82 parts, among them J301 Doepfer connector, J302 In_1, J303 In 2, J304 Out 1, J305 Out 2, J306 Out 1 Final, J307 Out 2 Final, U301 TL072, U302 TL072

Commit message: Update KicadJE_Counts2.sch
Parts:
- added D?: LED, AJ:LED_0805_2012Metric_Pad1.15x1.40mm_HandSolder, symbol Device:LED
- added R?: 10k, AJ:R_0805_AJ, symbol Device:R
Connections:
- net -12V: now also R?.1
- net GND: now also D?.2 (A)
- new net: D?.1 (K), R?.2
Changed lines of the file:
@@
 Wire Wire Line
 	1275 1000 2975 1000
+$Comp
+L Device:R R?
+U 1 1 5EC3116D
+P 1475 1850
+AR Path="/5CF11B19/5EC3116D" Ref="R?"  Part="1"
+AR Path="/5D4DB615/5EC3116D" Ref="R?"  Part="1"
+AR Path="/5D60ED9A/5EC3116D" Ref="R?"  Part="1"
+F 0 "R?" V 1475 1850 50  0000 C CNN
+F 1 "10k" V 1400 1825 50  0000 C CNN
+F 2 "AJ:R_0805_AJ" V 1405 1850 50  0001 C CNN
+F 3 "~" H 1475 1850 50  0001 C CNN
+	1    1475 1850
+	0    1    1    0
+$EndComp
+$Comp
+L Device:LED D?
+U 1 1 5EC3308B
+P 1200 1550
+F 0 "D?" V 1239 1432 50  0000 R CNN
+F 1 "LED" V 1148 1432 50  0000 R CNN
+F 2 "AJ:LED_0805_2012Metric_Pad1.15x1.40mm_HandSolder" H 1200 1550 50  0001 C CNN
+F 3 "~" H 1200 1550 50  0001 C CNN
+	1    1200 1550
+	0    -1   -1   0
+$EndComp
+Connection ~ 1200 1400
+Wire Wire Line
+	1200 1700 1200 1850
+Wire Wire Line
+	1200 1850 1325 1850
+Wire Wire Line
+	1625 1850 1675 1850
+Wire Wire Line
+	1675 1850 1675 1700
 $EndSCHEMATC

Commit message: Update KicadJE_Counts2.sch
Parts:
- RV301: value 100k_A4 -> 100k_1.1
- RV302: value 100k_A4 -> 100k_1.2
- RV303: value 100k_A4 -> 100k_2.1
- RV304: value 100k_A4 -> 100k_2.2
- gave numbers to parts that had none: 2
Connections:
- net POT1_C: now also RV301.2, RV301.3
- net POT1_L: now also RV301.1
- net POT2_C: now also RV302.2, RV302.3
- net POT2_L: now also RV302.1
- net POT3_C: no longer RV301.2, RV301.3
- net POT4_C: no longer RV302.2, RV302.3
- net POT4_L: no longer RV302.1
Changed lines of the file:
@@
 AR Path="/5D60ED9A/5F13A9C4" Ref="RV303"  Part="1"
 F 0 "RV303" V 2575 4550 50  0000 R CNN
-F 1 "100k_A4" V 2675 4575 50  0000 R CNN
+F 1 "100k_2.1" V 2675 4575 50  0000 R CNN
 F 2 "Potentiometer_THT:Potentiometer_China_RK09_Single_Vertical_AJ" H 2950 4400 50  0001 C CNN
 F 3 "~" H 2950 4400 50  0001 C CNN
@@
 AR Path="/5D60ED9A/5F31783B" Ref="RV304"  Part="1"
 F 0 "RV304" V 2575 5075 50  0000 R CNN
-F 1 "100k_A4" V 2675 5100 50  0000 R CNN
+F 1 "100k_2.2" V 2675 5100 50  0000 R CNN
 F 2 "Potentiometer_THT:Potentiometer_China_RK09_Single_Vertical_AJ" H 2950 4925 50  0001 C CNN
 F 3 "~" H 2950 4925 50  0001 C CNN
@@
 AR Path="/5D60ED9A/5F3F817E" Ref="RV301"  Part="1"
 F 0 "RV301" V 2575 2975 50  0000 R CNN
-F 1 "100k_A4" V 2675 3000 50  0000 R CNN
+F 1 "100k_1.1" V 2675 3000 50  0000 R CNN
 F 2 "Potentiometer_THT:Potentiometer_China_RK09_Single_Vertical_AJ" H 2950 2825 50  0001 C CNN
 F 3 "~" H 2950 2825 50  0001 C CNN
@@
 	1    0    0    1
 $EndComp
-Text HLabel 3250 2650 2    50   Input ~ 0
-POT3_H
-Text HLabel 3250 2825 2    50   Input ~ 0
-POT3_C
-Text HLabel 3250 3000 2    50   Input ~ 0
-POT3_L
-Text HLabel 3250 3200 2    50   Input ~ 0
-POT4_H
-Text HLabel 3250 3350 2    50   Input ~ 0
-POT4_C
-Text HLabel 3250 3500 2    50   Input ~ 0
-POT4_L
 $Comp
 L Device:R_POT RV?
@@
 AR Path="/5D60ED9A/5F3F818E" Ref="RV302"  Part="1"
 F 0 "RV302" V 2575 3500 50  0000 R CNN
-F 1 "100k_A4" V 2675 3525 50  0000 R CNN
+F 1 "100k_1.2" V 2675 3525 50  0000 R CNN
 F 2 "Potentiometer_THT:Potentiometer_China_RK09_Single_Vertical_AJ" H 2950 3350 50  0001 C CNN
 F 3 "~" H 2950 3350 50  0001 C CNN
@@
 AR Path="/5CF11B19/5EC3116D" Ref="R?"  Part="1"
 AR Path="/5D4DB615/5EC3116D" Ref="R?"  Part="1"
-AR Path="/5D60ED9A/5EC3116D" Ref="R?"  Part="1"
-F 0 "R?" V 1475 1850 50  0000 C CNN
+AR Path="/5D60ED9A/5EC3116D" Ref="R334"  Part="1"
+F 0 "R334" V 1475 1850 50  0000 C CNN
 F 1 "10k" V 1400 1825 50  0000 C CNN
 F 2 "AJ:R_0805_AJ" V 1405 1850 50  0001 C CNN
@@
 $EndComp
 $Comp
-L Device:LED D?
+L Device:LED D317
 U 1 1 5EC3308B
 P 1200 1550
-F 0 "D?" V 1239 1432 50  0000 R CNN
+F 0 "D317" V 1239 1432 50  0000 R CNN
 F 1 "LED" V 1148 1432 50  0000 R CNN
 F 2 "AJ:LED_0805_2012Metric_Pad1.15x1.40mm_HandSolder" H 1200 1550 50  0001 C CNN
@@
 Wire Wire Line
 	1675 1850 1675 1700
+Text HLabel 3250 2650 2    50   Input ~ 0
+POT1_H
+Text HLabel 3250 2825 2    50   Input ~ 0
+POT1_C
+Text HLabel 3225 3000 2    50   Input ~ 0
+POT1_L
+Text HLabel 3250 3200 2    50   Input ~ 0
+POT2_H
+Text HLabel 3250 3350 2    50   Input ~ 0
+POT2_C
+Text HLabel 3250 3500 2    50   Input ~ 0
+POT2_L
 $EndSCHEMATC
