File: KicadJE_Counts.sch (KiCad schematic (older format))
At the start: 19 parts, among them J101 In7, J102 In6, J103 In3, J104 Out10, J105 Out11, J106 Out9, J107 Out6, J108 Conn_02x03_Male

Commit message: cleanup old conn
Parts:
- removed J101: In7, AJ-Dropbox-Kicad:PJ301SM, symbol Connector:AudioJack2
- removed J102: In6, AJ-Dropbox-Kicad:PJ301SM, symbol Connector:AudioJack2
- removed J103: In3, AJ-Dropbox-Kicad:PJ301SM, symbol Connector:AudioJack2
- removed J104: Out10, AJ-Dropbox-Kicad:PJ301SM, symbol Connector:AudioJack2
- removed J105: Out11, AJ-Dropbox-Kicad:PJ301SM, symbol Connector:AudioJack2
- removed J106: Out9, AJ-Dropbox-Kicad:PJ301SM, symbol Connector:AudioJack2
- removed J107: Out6, AJ-Dropbox-Kicad:PJ301SM, symbol Connector:AudioJack2
- removed R101, R102, R103, R104, R105, R106: 10k, AJ:R_0805_AJ, symbol Device:R
Connections:
- net labels removed: A3, A6, A7, Out10Dist, Out11Dist, Out6Dist, Out9Dist
- wire segments 64 -> 26
Other:
- moved on the sheet: R109
